Commit message: jddhdhjd

File: foxy/SocialTech_ros2_ws/src/socialtech_challenge/urdf/camera.xacro (robot description, xacro)
@@ -16,5 +16,5 @@
 <link name="camera_link_optical"></link>
 <joint name="camera_optical_joint" type="fixed">
-    <origin xyz="0 0 0" rpy="-1.570796 0 -1.570796" />
+    <origin xyz="0 0 0" rpy="0 0 0" />
     <parent link="camera_link" />
     <child link="camera_link_optical" />

Commit message: funciona camara de percepcion

File: foxy/SocialTech_ros2_ws/src/socialtech_challenge/urdf/camera.xacro (robot description, xacro)
@@ -1,4 +1,5 @@
 <?xml version="1.0"?>
 <robot xmlns:xacro="http://www.ros.org/wiki/xacro">
+<xacro:property name="pi" value="3.1415926535897932" />
    <joint name="camera_joint" type="fixed">
     <parent link="base_link"/>
@@ -16,5 +17,5 @@
 <link name="camera_link_optical"></link>
 <joint name="camera_optical_joint" type="fixed">
-    <origin xyz="0 0 0" rpy="0 0 0" />
+    <origin xyz="0 0 0" rpy="${-pi/2} 0 ${-pi/2}" />
     <parent link="camera_link" />
     <child link="camera_link_optical" />
